File: dac.kicad_sch (KiCad schematic)
At the start: 62 parts, among them J10 AudioJack2_SwitchT, J11 AudioJack2_SwitchT, J12 AudioJack2_SwitchT, J13 AudioJack2_SwitchT, J7 AudioJack2_SwitchT, J8 AudioJack2_SwitchT, J9 AudioJack2_SwitchT, U3 TL074, U4 TL074

Commit message: Added initial layout.
Parts:
- removed R51, R52: 33k, Resistor_SMD:R_0805_2012Metric, symbol Device:R_Small
- added C48, C49: 100n, Capacitor_SMD:C_0805_2012Metric_Pad1.18x1.45mm_HandSolder, symbol Device:C_Small
- R16, R17, R18, R19, R20, R21, R22, R23, R24, R25, R26, R27, R28, R29, R30, R31, R32, R33, R34, R35, R36, R37, R38, R39, R40, R41, R42, R43, R44, R45, R46, R47, R48, R49, R50: footprint Resistor_SMD:R_0805_2012Metric -> Resistor_SMD:R_0805_2012Metric_Pad1.20x1.40mm_HandSolder
Connections:
- net GND: now also U4.12 (+), C48.1, C49.1; no longer U3.11 (V-), U4.11 (V-)
- net +3.3VA renamed +12V
- new net -12V: C48.2, C49.2, U3.11 (V-), U4.11 (V-)
Other:
- title: (none) -> STM32 Analog Breakout
- moved on the sheet: C39, C40
