File: lfo-nff.kicad_sch (KiCad schematic)
At the start: 0 parts

Commit message: Added initial layout.
Other:
- title: LFO NFF Test Board -> STM32 Analog Breakout
Changed lines of the file:
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@@
   (paper "A4")
   (title_block
-    (title "LFO NFF Test Board")
-    (date "2023-09-09")
-    (rev "1")
+    (title "STM32 Analog Breakout")
+    (date "2024-01-17")
+    (rev "A")
   )
   (sheet (at 92.71 27.94) (size 12.7 10.16) (fields_autoplaced)
