File: power.kicad_sch (KiCad schematic)
At the start: 18 parts, among them J14 Conn_02x05_Odd_Even, U5 R-78E3.3-1.0, U6 LM1117T-3.3, U7 LM4040B-10

Commit message: Added initial layout.
Parts:
- added J15, J16, J17, J18, J19: Conn_01x02, Connector_PinSocket_2.54mm:PinSocket_1x02_P2.54mm_Vertical, symbol Connector_Generic:Conn_01x02
- D3, D4: footprint Diode_SMD:D_SOD-323 -> Diode_SMD:D_SOD-323_HandSoldering
- R53, R54, R55: footprint Resistor_SMD:R_0805_2012Metric -> Resistor_SMD:R_0805_2012Metric_Pad1.20x1.40mm_HandSolder
- U6: footprint Package_TO_SOT_THT:TO-220-3_Horizontal_TabDown -> Package_TO_SOT_THT:TO-220-3_Vertical
Connections:
- net +12V: now also J18.1 (Pin_1); no longer C41.1, C43.1, C46.1, D3.1 (K), U5.1 (IN), U6.3 (VI)
- net +3.3V: now also J15.1 (Pin_1); no longer C42.1, D1.2 (A), U5.3 (OUT)
- net +3.3VA: now also J16.1 (Pin_1); no longer C44.1, D2.2 (A), U6.2 (VO)
- net -10V_Ref: now also J17.1 (Pin_1); no longer C45.2, R55.2, U7.2 (A)
- net -12V: now also J19.1 (Pin_1); no longer C47.2, D4.2 (A), R55.1
- new net: C45.2, J17.2 (Pin_2), R55.2, U7.2 (A)
- new net: C42.1, D1.2 (A), J15.2 (Pin_2), U5.3 (OUT)
- new net: C44.1, D2.2 (A), J16.2 (Pin_2), U6.2 (VO)
- new net +12V_Prejumper: C41.1, C43.1, C46.1, D3.1 (K), J18.2 (Pin_2), U5.1 (IN), U6.3 (VI)
- new net -12V_Prejumper: C47.2, D4.2 (A), J19.2 (Pin_2), R55.1
Other:
- title: (none) -> STM32 Analog Breakout
